Commit message: added two continuous wheels, front laser scan, and base_footprint; Add rviz config

File: my_rb1_description/urdf/my_rb1_robot.urdf (robot description, URDF)
Before this commit: robot rb1, 3 links, 2 joints
Links:
- added link base_footprint, mass 0
- added link front_laser, mass 1; collision cylinder length=0.05 radius=0.05; visual cylinder length=0.05 radius=0.05
- added link left_wheel, mass 1; collision cylinder length=0.025 radius=0.025; visual cylinder length=0.025 radius=0.025
- added link right_wheel, mass 1; collision cylinder length=0.025 radius=0.025; visual cylinder length=0.025 radius=0.025
- link base_link: mass 10 -> 20
Joints:
- added joint joint_base_footprint: type fixed, parent base_link, child base_footprint, origin xyz=0 0 -0.15 rpy=0 0 0
- added joint joint_laser_scan_chassis: type fixed, parent base_link, child front_laser, origin xyz=0.25 0 0.075 rpy=3.1415926 0 0
- added joint joint_left_wheel: type continuous, parent base_link, child left_wheel, origin xyz=0 -0.2 -0.15 rpy=0 0 0, axis 0 1 0, limit effort=10000 velocity=1000
- added joint joint_right_wheel: type continuous, parent base_link, child right_wheel, origin xyz=0 0.2 -0.15 rpy=0 0 0, axis 0 1 0, limit effort=10000 velocity=1000

Commit message: deleted bad urdf; optimized caster wheels size

File: my_rb1_description/urdf/my_rb1_robot.urdf (robot description, URDF)
Before this commit: robot rb1, 7 links, 6 joints
Links:
- link back_caster: geometry collision sphere radius=0.01; collision sphere radius=0.02
- link front_caster: geometry collision sphere radius=0.01; collision sphere radius=0.02

Commit message: Added gazebo plugins for differential drive and laser scan; Tested with rostopic

File: my_rb1_description/urdf/my_rb1_robot.urdf (robot description, URDF)
Before this commit: robot rb1, 7 links, 6 joints
Joints:
- removed joint joint_laser_scan_chassis
- added joint joint_front_laser_base_link: type fixed, parent base_link, child front_laser, origin xyz=0.25 0 0.075 rpy=3.1415926 0 0

Commit message: Optimized laser mass and intertia; add mass to base_footprint

File: my_rb1_description/urdf/my_rb1_robot.urdf (robot description, URDF)
Before this commit: robot rb1, 7 links, 6 joints
Links:
- link base_footprint: mass 0 -> 0.5
- link front_laser: mass 1 -> 0.5

Commit message: Added <mu> tags

File: my_rb1_description/urdf/my_rb1_robot.urdf (robot description, URDF)
Before this commit: robot rb1, 7 links, 6 joints
Links:
- link base_footprint: mass 0.5 -> 0
- link front_laser: mass 0.5 -> 0
